Commit message: cam added

File: road100_description/urdf/road100.urdf (robot description, URDF)
Before this commit: robot rlcar, 9 links, 8 joints
Links:
- added link camera_link, mass 0.01; collision sphere radius=0.01
Joints:
- added joint camera_joint: type fixed, parent base_link, child camera_link, origin xyz=0.08 0 0.045 rpy=0 0 0
