Commit message: ignition till rviz done

File: road100_ignition/urdf/gz.xacro (robot description, xacro)
@@ -69,25 +69,23 @@
 </gazebo>
 <!-- ........................... CAMERA config ................................... -->
-<!-- <xacro:if value="$(arg camera_enabled)">
-    <gazebo reference="kinect_camera">
-        <sensor type="depth_camera" name="kinect_camera">
-            <update_rate>30.0</update_rate>
-            <topic>kinect_camera</topic>
-            <ignition_frame_id>kinect_camera</ignition_frame_id>
-            <camera_info_topic>camera_info</camera_info_topic>
-            <camera>
-                <horizontal_fov>${radians(camera_horizontal_fov)}</horizontal_fov>
-                <image>
-                    <width>640</width>
-                    <height>480</height>
-                    <format>R8G8B8</format>
-                </image>
-                <clip>
-                    <near>0.05</near>
-                    <far>8.0</far>
-                </clip>
-            </camera>
-        </sensor>
-    </gazebo>
-</xacro:if> -->
+<gazebo reference="camera_link">
+    <sensor name="camera" type="camera">
+        <camera>
+            <horizontal_fov>1.047</horizontal_fov>
+            <image>
+                <width>640</width>
+                <height>480</height>
+                <format>R8G8B8</format>
+            </image>
+            <clip>
+                <near>0.05</near>
+                <far>8.0</far>
+            </clip>
+        </camera>
+        <always_on>1</always_on>
+        <update_rate>30</update_rate>
+        <visualize>true</visualize>
+        <topic>camera</topic>
+    </sensor>
+</gazebo>
 </robot>

File: road100_ignition/urdf/road100.urdf.xacro (robot description, xacro)
@@ -155,3 +155,20 @@
     <child link="lidar_link"/>
   </joint>
+  <link name="camera_link">
+    <inertial>
+      <mass value="0.01"/>
+      <inertia ixx="0.00004" ixy="0" ixz="0" iyy="0.00004" iyz="0" izz="0.00004"/>
+    </inertial>
+    <collision>
+      <origin rpy="0 0 0" xyz="0 0 0"/>
+      <geometry>
+        <sphere radius="0.01"/>
+      </geometry>
+    </collision>
+  </link>
+  <joint name="camera_joint" type="fixed">
+    <origin xyz="0.08 0 0.045" rpy="0 0 0"/>
+    <parent link="base_link"/>
+    <child link="camera_link"/>
+  </joint>
 </robot>
